File: KiCad/tester/7SegTester.kicad_sch (KiCad schematic)
At the start: 11 parts, among them J1 Conn_01x08_Pin

Commit message: resistors, footprints, and org
Parts:
- added RN1: R_Pack08, Package_DIP:DIP-16_W7.62mm_Socket, symbol Device:R_Pack08
- 7SEG1: footprint Display_7Segment:D1X8K -> footprints:LS-5161AS
Connections:
- net A: now also RN1.8 (R8.1); no longer SR1.15 (QA)
- net B: now also RN1.1 (R1.1); no longer SR1.1 (QB)
- net C: now also RN1.2 (R2.1); no longer SR1.2 (QC)
- net D: now also RN1.3 (R3.1); no longer SR1.3 (QD)
- net D5: now also SR1.11 (SRCLK); no longer SR1.12 (RCLK)
- net D7: now also SR1.14 (SER); no longer SR1.11 (SRCLK)
- net DP: now also RN1.7 (R7.1); no longer SR1.7 (QH)
- net E: now also RN1.4 (R4.1); no longer SR1.4 (QE)
- net F: now also RN1.5 (R5.1); no longer SR1.5 (QF)
- net G: now also RN1.6 (R6.1); no longer SR1.6 (QG)
- net D8 renamed PWM8
- net PWM8: now also R3.1; no longer SR1.14 (SER)
- net PWM6 renamed D6
- net D6: now also SR1.12 (RCLK); no longer R3.1
- new net: RN1.13 (R4.2), SR1.4 (QE)
- new net: RN1.14 (R3.2), SR1.3 (QD)
- new net: RN1.15 (R2.2), SR1.2 (QC)
- new net: RN1.16 (R1.2), SR1.1 (QB)
- new net: RN1.9 (R8.2), SR1.15 (QA)
- new net 10: RN1.10 (R7.2), SR1.7 (QH)
- new net 11: RN1.11 (R6.2), SR1.6 (QG)
- new net 12: RN1.12 (R5.2), SR1.5 (QF)
Other:
- moved on the sheet: SR1
